File: Electronics/CapacitorSensor/Proto-3/P3R1/P3R1.kicad_pcb (KiCad board)
At the start: 2 copper layers, 100 x 100 mm, 164 parts, among them Q1 BC547, Q10 BS107, Q11 BS107, Q12 BS107, Q13 BS107, Q14 BS107, Q15 BS107, Q16 BS107, Q17 BC547, Q18 BC547, Q19 BC547, Q2 BC547, Q20 BC547, Q21 BC547, Q22 BC547, Q23 BC547, Q24 BC547, Q3 BC547, Q4 BC547, Q5 BC547, Q6 BC547, Q7 BC547, Q8 BC547, Q9 BS107, U1 TC2185-2.8VxCTTR, U10 LM318N, U11 LM319, U12 LM319, U13 LM319, U14 LM319, U15 74LS14, U16 74LS14, U17 74LS14, U18 LM339, U19 LM339, U2 AMS1117-5.0, U20 STM32H725IET6, U3 LM318N, U4 LM318N, U5 LM318N, U6 LM318N, U7 LM318N, U8 LM318N, U9 LM318N

Commit message: Moare
Parts:
- added U21: 74LS14, Package_SO:SOIC-14_3.9x8.7mm_P1.27mm, F.Cu at (129.1, 16.1)
- added U22: LM393, Package_SO:SOIC-8_3.9x4.9mm_P1.27mm, F.Cu at (137.5, 20.6)
- added U23: LM393, Package_SO:SOIC-8_3.9x4.9mm_P1.27mm, F.Cu at (145.9, 20.6)
- added U24: LM393, Package_SO:SOIC-8_3.9x4.9mm_P1.27mm, F.Cu at (145.9, 14.2)
- added U25: LM393, Package_SO:SOIC-8_3.9x4.9mm_P1.27mm, F.Cu at (137.5, 14.2)
- added U26: STM32L431RCTx, Package_QFP:LQFP-64_10x10mm_P0.5mm, F.Cu at (132.1, 37.3)
- added U27: STM32L431RCTx, Package_QFP:LQFP-64_10x10mm_P0.5mm, F.Cu at (162.9, 18.2)
- U10, U3, U4, U5, U6, U7, U8, U9: footprint Package_DIP:DIP-8-16_W7.62mm_Socket -> Package_SO:SOIC-8_3.9x4.9mm_P1.27mm
- U11, U12, U13, U14: value LM319 -> LM318N; footprint Package_SO:SOIC-14-16_3.9x9.9mm_P1.27mm -> Package_SO:SOIC-8_3.9x4.9mm_P1.27mm
- U15, U16, U17: value 74LS14 -> LM318N; footprint Package_SO:SOIC-14-16_3.9x9.9mm_P1.27mm -> Package_SO:SOIC-8_3.9x4.9mm_P1.27mm
- U18: value LM339 -> LM318N; footprint Package_SO:SOIC-14-16_3.9x9.9mm_P1.27mm -> Package_SO:SOIC-8_3.9x4.9mm_P1.27mm
- U19: value LM339 -> 74LS14; footprint Package_SO:SOIC-14-16_3.9x9.9mm_P1.27mm -> Package_SO:SOIC-14_3.9x8.7mm_P1.27mm
- U20: value STM32H725IET6 -> 74LS14; footprint Package_QFP:LQFP-176_24x24mm_P0.5mm -> Package_SO:SOIC-14_3.9x8.7mm_P1.27mm
Connections:
- Q17 pad 3: Net-(C9-Pad1) -> B0
- Q18 pad 3: Net-(C10-Pad1) -> B1
- Q19 pad 3: Net-(C11-Pad1) -> B2
- Q20 pad 3: Net-(C12-Pad1) -> B3
- Q21 pad 3: Net-(C13-Pad1) -> B4
- Q22 pad 3: Net-(C14-Pad1) -> B5
- Q23 pad 3: Net-(C15-Pad1) -> B6
- Q24 pad 3: Net-(C16-Pad1) -> B7
- U11 pad 3: B0 -> Net-(R65-Pad1)
- U11 pad 4: Net-(R65-Pad1) -> B0
- U11 pad 5: Net-(R57-Pad2) -> unconnected-(U11-Pad5)
- U11 pad 6: (no net) -> Net-(D17-Pad2)
- U11 pad 7: Net-(D18-Pad2) -> VCC
- U11 pad 8: B1 -> unconnected-(U11-Pad8)
- U12 pad 3: B2 -> Net-(R66-Pad1)
- U12 pad 4: Net-(R67-Pad1) -> B1
- U12 pad 5: Net-(R59-Pad2) -> unconnected-(U12-Pad5)
- U12 pad 6: (no net) -> Net-(D18-Pad2)
- U12 pad 7: Net-(D20-Pad2) -> VCC
- U12 pad 8: B3 -> unconnected-(U12-Pad8)
- U13 pad 3: B4 -> Net-(R67-Pad1)
- U13 pad 4: Net-(R69-Pad1) -> B2
- U13 pad 5: Net-(R61-Pad2) -> unconnected-(U13-Pad5)
- U13 pad 6: (no net) -> Net-(D19-Pad2)
- U13 pad 7: Net-(D22-Pad2) -> VCC
- U13 pad 8: B5 -> unconnected-(U13-Pad8)
- U14 pad 3: B6 -> Net-(R68-Pad1)
- U14 pad 4: Net-(R71-Pad1) -> B3
- U14 pad 5: Net-(R63-Pad2) -> unconnected-(U14-Pad5)
- U14 pad 6: (no net) -> Net-(D20-Pad2)
- U14 pad 7: Net-(D24-Pad2) -> VCC
- U14 pad 8: B7 -> unconnected-(U14-Pad8)
- U15 pad 1: Net-(D17-Pad2) -> unconnected-(U15-Pad1)
- U15 pad 3: Net-(U15-Pad2) -> Net-(R69-Pad1)
- U15 pad 4: Q0 -> B4
- U15 pad 5: Net-(D18-Pad2) -> unconnected-(U15-Pad5)
- U15 pad 6: Net-(U15-Pad6) -> Net-(D21-Pad2)
- U15 pad 7: (no net) -> VCC
- U15 pad 8: Q1 -> unconnected-(U15-Pad8)
- U16 pad 1: Net-(D20-Pad2) -> unconnected-(U16-Pad1)
- U16 pad 3: Net-(U16-Pad2) -> Net-(R70-Pad1)
- U16 pad 4: Q3 -> B5
- U16 pad 5: Net-(D21-Pad2) -> unconnected-(U16-Pad5)
- U16 pad 6: Net-(U16-Pad6) -> Net-(D22-Pad2)
- U16 pad 7: (no net) -> VCC
- U16 pad 8: Q4 -> unconnected-(U16-Pad8)
- U17 pad 1: Net-(D23-Pad2) -> unconnected-(U17-Pad1)
- U17 pad 3: Net-(U17-Pad2) -> Net-(R71-Pad1)
- U17 pad 4: Q6 -> B6
- U17 pad 5: Net-(D24-Pad2) -> unconnected-(U17-Pad5)
- U17 pad 6: Net-(U17-Pad6) -> Net-(D23-Pad2)
- U17 pad 7: (no net) -> VCC
- U17 pad 8: Q7 -> unconnected-(U17-Pad8)
- U18 pad 3: unconnected-(U18-Pad3) -> Net-(R72-Pad1)
- U18 pad 4: unconnected-(U18-Pad4) -> B7
- U18 pad 6: unconnected-(U18-Pad6) -> Net-(D24-Pad2)
- U18 pad 7: unconnected-(U18-Pad7) -> VCC
- U19 pad 1: unconnected-(U19-Pad1) -> Net-(D17-Pad2)
- U19 pad 10: unconnected-(U19-Pad10) -> Net-(U19-Pad10)
- U19 pad 11: unconnected-(U19-Pad11) -> Net-(D19-Pad2)
- U19 pad 12: unconnected-(U19-Pad12) -> Q2
- U19 pad 14: unconnected-(U19-Pad14) -> (no net)
- U19 pad 3: unconnected-(U19-Pad3) -> Net-(U19-Pad2)
- U19 pad 4: unconnected-(U19-Pad4) -> Q0
- U19 pad 5: unconnected-(U19-Pad5) -> Net-(D18-Pad2)
- U19 pad 6: unconnected-(U19-Pad6) -> Net-(U19-Pad6)
- U19 pad 7: unconnected-(U19-Pad7) -> (no net)
- U19 pad 8: unconnected-(U19-Pad8) -> Q1
- U19 pad 9: unconnected-(U19-Pad9) -> Net-(U19-Pad6)
- U20 pad 1: unconnected-(U20-Pad1) -> Net-(D20-Pad2)
- U20 pad 10: unconnected-(U20-Pad10) -> Net-(U20-Pad10)
- U20 pad 11: unconnected-(U20-Pad11) -> Net-(D22-Pad2)
- U20 pad 12: unconnected-(U20-Pad12) -> Q5
- U20 pad 13: unconnected-(U20-Pad13) -> Net-(U20-Pad10)
- U20 pad 14: unconnected-(U20-Pad14) -> (no net)
- U20 pad 2: unconnected-(U20-Pad2) -> Net-(U20-Pad2)
- U20 pad 3: unconnected-(U20-Pad3) -> Net-(U20-Pad2)
- U20 pad 4: unconnected-(U20-Pad4) -> Q3
- U20 pad 5: unconnected-(U20-Pad5) -> Net-(D21-Pad2)
- U20 pad 6: unconnected-(U20-Pad6) -> Net-(U20-Pad6)
- U20 pad 7: unconnected-(U20-Pad7) -> (no net)
- U20 pad 8: unconnected-(U20-Pad8) -> Q4
- U20 pad 9: unconnected-(U20-Pad9) -> Net-(U20-Pad6)
- U3 pad 8: Net-(C9-Pad1) -> Net-(C17-Pad1)
